File: pcb/sous-vide.sch (KiCad schematic (older format))
At the start: 19 parts, among them J1 Screw_Terminal_01x02, J2 Conn_ARM_JTAG_SWD_10, SW1 SW_Push, SW2 SW_SPDT, SW3 Rotary_Encoder_Switch, U1 HLK-PM03, U2 LM1117-3.3, U3 STM32F030F4Px

Commit message: Completing schematic
Parts:
- removed C3: 4.7uF, symbol Passive:CAP
- removed D1: D_Schottky, symbol Device:D_Schottky
- removed J2: Conn_ARM_JTAG_SWD_10, Connector_PinHeader_1.27mm:PinHeader_2x05_P1.27mm_Vertical_SMD, symbol Connector:Conn_ARM_JTAG_SWD_10
- removed SW2: SW_SPDT, symbol Switch:SW_SPDT
- added D?: PWR, symbol Device:LED
- added K? (x2): SANYOU_SRD_Form_C, Relay_THT:Relay_SPDT_SANYOU_SRD_Series_Form_C, symbol Relay:SANYOU_SRD_Form_C
- added P?: HEADER_1x3, symbol header:HEADER_1x3
- added P?: DS18B20_TempSens, symbol header:HEADER_1x3
- added P?: ISP, symbol header:HEADER_1x4
- added P?: SWD, symbol header:HEADER_1x4
- added P?: BOOT_JMP, symbol header:HEADER_1x2
- added P?: HEADER_1x4, symbol header:HEADER_1x4
- added R?: 560, symbol Device:R
- added R? (x2): 4.7K, symbol Device:R
- added R?: 1K, symbol Device:R
- added RV?: 10K, symbol Device:R_POT
- added S?: SPDT, symbol Electromechanical:SWITCH_ROCKER_SPDT_ON_ON
- added U?: NHD-0420H1Z, Display:NHD-0420H1Z, symbol Display_Character:NHD-0420H1Z
- C1: value CAPP -> 22uF
- C2: value CAPP -> 10uF
- C4: value 4.7uF -> 100nF
- F1: value Fuse -> 200mA Slow Fuse
- F2: value Fuse -> 72C Thermal Fuse
- F3: value Fuse -> 630mA Quick Fuse
- SW1: value SW_Push -> SW_RST
- U1: value HLK-PM03 -> HLK-PM05
Connections:
- net GND: now also C1.2, C2.2, C5.1, D?.1 (K), P?.2 (P2), P?.3 (P3), P?.4 (P4), P?.4 (P4), RV?.1, U?.1 (VSS), U?.16 (K); no longer C1.1, C2.1, C5.2
- net SWDCLK: now also P?.3 (P3)
- net SWDIO: now also P?.2 (P2)
- net VCC: now also C5.2, R1.2, SW1.2, U3.4 (NRST), P?.1 (P1), P?.1 (P1), P?.1 (P1), R?.1, R?.2
- net VPP: now also C1.1, C2.1, U2.3 (VI), R?.1, U?.15 (A), U?.2 (VDD); no longer C1.2, C2.2
- net at RV1.1, U1.1 (L1): now also S?.3 (B); no longer J1.2 (Pin_2)
- net at R1.1: now also P?.1 (P1), R?.2; no longer U3.1 (BOOT0)
- net TX: now reaches U3.17 (PA9)
- net TX: now also P?.3 (P3)
- net RX: now reaches U3.18 (PA10)
- net RX: now also P?.2 (P2)
- removed net RST: C5.1, SW1.2, U3.4 (NRST)
- new net: J1.2 (Pin_2), S?.2 (COM)
- new net: RV?.2, U?.3 (VO)
- new net: D?.2 (A), R?.2
- new net: R?.2, RV?.3
- new net BOOT0: R?.1, U3.1 (BOOT0)
- new net TMPSS: P?.2 (P2), R?.1
Other:
- moved on the sheet: C1, C2, C4, C5, F1, F2, F3, J1, R1, RV1, SW1, U1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
